File: kicad_ble/kicad_ble.kicad_pcb (KiCad board)
At the start: 2 copper layers, 207.8 x 60.2 mm, 94 parts, among them J2 78171-0002, J3 TC2030_SWD, SW1 RST, SW2 RotaryEncoder_Switch, U1 MAX17048, U2 BQ24075, U3 SRV05-4, U4 nRF52840_E73-2G4M08S1C, U5 74LVC1G11, Y1 32.768 KHz

Commit message: first 'finished' version
Parts:
- added J1: TC2030_SWD, Connector_PinHeader_2.54mm:PinHeader_1x05_P2.54mm_Vertical, F.Cu at (62.9, 99.1)
Connections:
- H1 pad 1: GND -> unconnected-(H1-Pad1)
- H2 pad 1: GND -> unconnected-(H2-Pad1)
- H3 pad 1: GND -> unconnected-(H3-Pad1)
- H4 pad 1: GND -> unconnected-(H4-Pad1)
- J2 pad MP: unconnected-(J2-MountPin-PadMP) -> connect_me_if_you_wish
- U4 pad 10: unconnected-(U4-P0.30/AIN6-Pad10) -> c7
- U4 pad 12: r0 -> c8
- U4 pad 14: r1 -> r0
- U4 pad 16: unconnected-(U4-P0.08-Pad16) -> r1
- U4 pad 4: c7 -> ENC_DP
- U4 pad 41: unconnected-(U4-P0.09/NFC1-Pad41) -> c9
- U4 pad 6: unconnected-(U4-P1.13-Pad6) -> c5
- U4 pad 9: unconnected-(U4-P0.31/AIN7-Pad9) -> c6
Routing:
- net c5: track 98.7 -> 146.4 mm, vias 0 -> 4
- net ENC_DP: track 39.8 -> 86.3 mm, vias 0 -> 2
- net c9: track 185.3 -> 229.4 mm, vias 1 -> 4
- net c8: track 156.0 -> 191.1 mm, vias 0 -> 2
- net c6: track 112.1 -> 146.9 mm, vias 0 -> 2
- net c7: track 146.5 -> 180.2 mm, vias 0 -> 2
- net SWDCLK: track 55.4 -> 84.8 mm
- net c4: track 77.8 -> 66.0 mm
- net GND: track 163.2 -> 171.4 mm, vias 45 -> 48
- net RST: track 57.0 -> 63.5 mm, vias 2 -> 3
- net VDD: track 80.3 -> 86.2 mm
- net r2: track 233.2 -> 227.4 mm
- net SWDIO: track 63.5 -> 68.3 mm
- net Net-(D13-A1): track 17.2 -> 21.7 mm, vias 0 -> 1
- net D+: track 110.7 -> 107.2 mm
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- added copper zone on F.Cu, net connect_me_if_you_wish
Other:
- outline, holes or cut-outs redrawn

Commit message: next iteration
Parts:
- added G***: LOGO, projectlib:tsuru, F.Cu at (81.2, 97.3)
- added J4: solder_me+, Connector_Pin:Pin_D0.7mm_L6.5mm_W1.8mm_FlatFork, F.Cu at (135.5, 98.8)
- added J5: solder_me-, Connector_PinHeader_2.54mm:PinHeader_1x01_P2.54mm_Vertical, F.Cu at (135.5, 103.4)
- J1: value TC2030_SWD -> thts
- J2: value 78171-0002 -> JST-GH; footprint PCM_marbastlib-various:Molex_Pico-EZmate_78171-0002_1x02-1MP_P1.20mm_Vertical -> Connector_JST:JST_GH_SM02B-GHS-TB_1x02-1MP_P1.25mm_Horizontal
- moved J2 7.08 mm to (129.9, 102.6), turned to -135 degrees
- moved C14 5.36 mm to (72.7, 105.3)
- moved C4 5.36 mm to (106.7, 109.0)
- moved C6 5.36 mm to (115.0, 106.2)
- moved C8 5.36 mm to (113.4, 109.0)
- moved D13 5.36 mm to (144.7, 110.6)
- moved D8 5.36 mm to (144.7, 107.2)
- moved H4 5.36 mm to (245.9, 105.3)
- moved LED1 5.36 mm to (56.0, 105.3)
- moved MX23 5.36 mm to (87.5, 114.8)
- moved MX24 5.36 mm to (106.6, 114.8)
- moved MX25 5.36 mm to (125.6, 114.8)
- moved MX26 5.36 mm to (163.7, 114.8)
- moved MX27 5.36 mm to (182.8, 114.8)
- moved MX29 5.36 mm to (220.9, 114.8)
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Connections:
- J2 pad MP: connect_me_if_you_wish -> unconnected-(J2-MountPin-PadMP)
Routing:
- net c7: track 180.2 -> 192.2 mm
- net +BATT: track 18.0 -> 26.1 mm, vias 0 -> 1
- net +5V: track 101.9 -> 94.2 mm
- net GND: track 171.4 -> 173.6 mm
- net Net-(D13-A1): track 21.7 -> 20.3 mm
- removed copper zone on F.Cu, net connect_me_if_you_wish
Other:
- outline, holes or cut-outs redrawn
- board text added: "Call me maybe!"
- board text added: "陰 極"
- board text added: "陽 極"
- board text added: "電 池"
- board text removed: "Hope your fix is going well!"
