File: kicad_ble/kicad_ble.kicad_sch (KiCad schematic)
At the start: 93 parts, among them J2 78171-0002, J3 TC2030_SWD, SW1 RST, SW2 RotaryEncoder_Switch, U1 MAX17048, U2 BQ24075, U3 SRV05-4, U4 nRF52840_E73-2G4M08S1C, U5 74LVC1G11, Y1 32.768 KHz

Commit message: first 'finished' version
Parts:
- added J3: TC2030_SWD, Connector_PinHeader_2.54mm:PinHeader_1x05_P2.54mm_Vertical, symbol Connector_Generic:Conn_01x05
Connections:
- net ENC_DP: now also U4.4 (P0.28/AIN4)
- net GND: now also J3.1 (Pin_1); no longer H1.1, H2.1, H3.1, H4.1
- net RST: now also J3.3 (Pin_3)
- net SWDCLK: now also J3.4 (Pin_4)
- net SWDIO: now also J3.2 (Pin_2)
- net VDD: now also J3.5 (Pin_5)
- net c5: now also U4.6 (P1.13)
- net c6: now also U4.9 (P0.31/AIN7)
- net c7: now also U4.10 (P0.30/AIN6); no longer U4.4 (P0.28/AIN4)
- net c8: now also U4.12 (P0.26)
- net c9: now also U4.41 (P0.09/NFC1)
- net r0: now also U4.14 (P0.06); no longer U4.12 (P0.26)
- net r1: now also U4.16 (P0.08); no longer U4.14 (P0.06)
- net connect_me_if_you_wish: now reaches J2.MP (MountPin)
- no-connect marks 12 -> 14
Other:
- note added: "THT programming option"

Commit message: next iteration
Parts:
- added J4: solder_me+, Connector_Pin:Pin_D0.7mm_L6.5mm_W1.8mm_FlatFork, symbol Connector_Generic:Conn_01x01
- added J5: solder_me-, Connector_PinHeader_2.54mm:PinHeader_1x01_P2.54mm_Vertical, symbol Connector_Generic:Conn_01x01
- J2: value 78171-0002 -> JST-GH; footprint PCM_marbastlib-various:Molex_Pico-EZmate_78171-0002_1x02-1MP_P1.20mm_Vertical -> Connector_JST:JST_GH_SM02B-GHS-TB_1x02-1MP_P1.25mm_Horizontal
- J3: value TC2030_SWD -> thts; now left out of the parts list
Connections:
- net +BATT: now also J4.1 (Pin_1)
- net GND: now also J5.1 (Pin_1)
- net connect_me_if_you_wish: no longer names the net of J2.MP (MountPin)
- no-connect marks 14 -> 15
Other:
- moved on the sheet: C4, C5, C7, C8, J2, J3
